File: KiCad/miniParMain.kicad_pcb (KiCad board)
At the start: 4 copper layers, 25 x 40 mm, 30 parts, among them J2 USB_C_Receptacle, J4 Conn_01x02_Pin, J5 secondBoard, SW2 SW_Push, U1 AS7341-DLGT, U2 IP4234CZ6, U5 AP7312-1833W6-7, U8 ESP8685, Y2 40MHz

Commit message: add bme to PCB - update the casing
Parts:
- added C5: 2.2u, Capacitor_SMD:C_0603_1608Metric_Pad1.08x0.95mm_HandSolder, F.Cu at (107.0, 103.8)
- added C7: 2.2u, Capacitor_SMD:C_0603_1608Metric_Pad1.08x0.95mm_HandSolder, F.Cu at (108.9, 103.8)
- added C8: 2.2u, Capacitor_SMD:C_0603_1608Metric_Pad1.08x0.95mm_HandSolder, F.Cu at (89.8, 100.0)
- added R14: 5.1K, Resistor_SMD:R_0603_1608Metric, F.Cu at (110.5, 103.7)
- added U3: BME280, Package_LGA:Bosch_LGA-8_2.5x2.5mm_P0.65mm_ClockwisePinNumbering, F.Cu at (108.0, 100.0)
- added U9: LIS2DE12, Package_LGA:LGA-12_2x2mm_P0.5mm, F.Cu at (92.0, 100.0)
Routing:
- net SCL: track 26.4 -> 44.6 mm, vias 3 -> 4
- net V+3V: track 28.0 -> 44.6 mm, vias 9 -> 14
- net GND: track 35.7 -> 51.2 mm, vias 53 -> 63
- net SDA: track 29.5 -> 42.0 mm, vias 3 -> 5
- net Net-(U3-SDO): track 0.00 -> 2.48 mm
Other:
- board text added: "simplePAR V1.2"
- board text removed: "miniPAR V1.1"
