File: KiCad/miniParMain.kicad_sch (KiCad schematic)
At the start: 37 parts, among them J1 Conn_01x08, J2 USB_C_Receptacle, J4 Conn_01x02_Pin, J5 secondBoard, SW2 SW_Push, U1 AS7341-DLGT, U2 IP4234CZ6, U5 AP7312-1833W6-7, U8 ESP8685, Y2 40MHz

Commit message: add bme to PCB - update the casing
Parts:
- added C5, C7, C8: 2.2u, Capacitor_SMD:C_0603_1608Metric_Pad1.08x0.95mm_HandSolder, symbol Device:C
- added R14: 5.1K, Resistor_SMD:R_0603_1608Metric, symbol main-rescue:R-
- added U3: BME280, Package_LGA:Bosch_LGA-8_2.5x2.5mm_P0.65mm_ClockwisePinNumbering, symbol Sensor:BME280
- added U9: LIS2DE12, Package_LGA:LGA-12_2x2mm_P0.5mm, symbol Sensor_Motion:LIS2DE12
Connections:
- net GND: now also C5.2, C7.2, C8.2, U3.1 (GND), U3.7 (GND), U9.3 (SA0/SDO), U9.5 (RES), U9.6 (GND), U9.7 (GND), U9.8 (GND)
- net SCL: now also U3.4 (SCK), U9.1 (SCL/SPC)
- net SDA: now also U3.3 (SDI), U9.4 (SDA/SDI)
- net V+3V: now also C5.1, C7.1, C8.1, R14.2, U3.2 (CSB), U3.6 (VDDIO), U3.8 (VDD), U9.10 (Vdd_IO), U9.2 (~{CS}), U9.9 (Vdd)
- new net: R14.1, U3.5 (SDO)
- new net INT_1: U9.12 (INT1)
- new net INT_2: U9.11 (INT2)
Other:
- moved on the sheet: J4, J5, R12, R29, R3, R30, R6, R7, R8, SW2
